File: schematic.kicad_sch (KiCad schematic)
At the start: 39 parts, among them J3 USB_C_Receptacle_USB2.0_16P

Commit message: v1.0.0: Update title block, add project version variable
Other:
- title: (none) -> Prowler Keyboard
Changed lines of the file:
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@@
 	(generator_version "8.0")
 	(paper "A4")
+	(title_block
+		(title "Prowler Keyboard")
+		(date "2024-12-17")
+		(rev "${VER}")
+	)
 	(junction
 		(at 15.24 24.13)
