File: switch.kicad_sch (KiCad schematic)
At the start: 3 parts

Commit message: v1.0.0: Update title block, add project version variable
Other:
- title: (none) -> Prowler Keyboard
Changed lines of the file:
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@@
 	(generator_version "8.0")
 	(paper "A4")
+	(title_block
+		(title "Prowler Keyboard")
+		(date "2024-12-17")
+		(rev "${VER}")
+	)
 	(hierarchical_label "V_LED"
 		(shape passive)
